Commit message: Actualizacion README 07-URDF y exportacion URDF (BaseFija / JointCremallera)
README con el proceso de exportacion desde SolidWorks (SW2URDF), anatomia del
URDF y relacion con la tabla DH, validacion con PyBullet/yourdfpy. Se reemplaza
la exportacion del 18-jun por la del 9-jul y se corrigen URDF.py y URDFMOV.py
(rutas relativas, posicion real del efector).

File: 7. URDF/ArchivosURDF/urdf/EnsamblajeFinal.SLDASM.urdf (robot description, URDF)
Before this commit: robot EnsamblajeFinal.SLDASM, 4 links, 3 joints
Links:
- removed link Parte1
- added link BaseFija, mass 1.2446; collision mesh filename=package://EnsamblajeFinal.SLDASM/meshes/BaseFija.STL; visual mesh filename=package://EnsamblajeFinal.SLDASM/meshes/BaseFija.STL
Joints:
- removed joint JointC
- added joint JointCremallera: type prismatic, parent Parte3, child Cremallera, origin xyz=0.1619 0 0.0041 rpy=-3.1416 0 0, axis 0 0 1, limit lower=0 upper=0.054 effort=10 velocity=0.1
- joint JointP2: limit lower=-1.5708 upper=1.5708 effort=10 velocity=1.0 -> (none); parent Parte1 -> BaseFija; type revolute -> continuous
- joint JointP3: limit lower=-1.5708 upper=1.5708 effort=10 velocity=1.0 -> (none); type revolute -> continuous
